File: SofleKeyboard.kicad_sch (KiCad schematic)
At the start: 83 parts, among them J3 OLED, SW1 SW_PUSH_LED, SW10 SW_PUSH_LED, SW11 SW_PUSH_LED, SW12 SW_PUSH_LED, SW13 SW_PUSH_LED, SW14 SW_PUSH_LED, SW15 SW_PUSH_LED, SW16 SW_PUSH_LED, SW17 SW_PUSH_LED, SW18 SW_PUSH_LED, SW19 SW_PUSH_LED, SW2 SW_PUSH_LED, SW20 SW_PUSH_LED, SW21 SW_PUSH_LED, SW22 SW_PUSH_LED, SW23 SW_PUSH_LED, SW24 SW_PUSH_LED, SW26 SW_PUSH_LED, SW27 SW_PUSH_LED, SW28 SW_PUSH_LED, SW29 SW_PUSH_LED, SW3 SW_PUSH_LED, SW30 SW_PUSH_LED, SW4 SW_PUSH_LED, SW5 SW_PUSH_LED, SW6 SW_PUSH_LED, SW7 SW_PUSH_LED, SW8 SW_PUSH_LED, SW9 SW_PUSH_LED, U1 ProMicro

Commit message: some stuff
Parts:
- added D25: 1N4148W, Diode_SMD:D_SOD-123, symbol Diode:1N4148W
Connections:
- net row1: now also D25.1 (K); no longer SW_NAV_1.3
- new net: D25.2 (A), SW_NAV_1.3
Changed lines of the file:
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@@
 	(wire
 		(pts
+			(xy 64.77 149.86) (xy 66.04 149.86)
+		)
+		(stroke
+			(width 0)
+			(type default)
+		)
+	)
+	(wire
+		(pts
 			(xy 213.36 92.71) (xy 233.68 92.71)
 		)
@@
 	(wire
 		(pts
-			(xy 62.23 149.86) (xy 66.04 149.86)
-		)
-		(stroke
-			(width 0)
-			(type default)
-		)
-	)
-	(wire
-		(pts
 			(xy 172.72 76.2) (xy 152.4 76.2)
 		)
@@
 	(wire
 		(pts
+			(xy 54.61 149.86) (xy 57.15 149.86)
+		)
+		(stroke
+			(width 0)
+			(type default)
+		)
+	)
+	(wire
+		(pts
 			(xy 31.75 101.6) (xy 36.83 101.6)
 		)
@@
 	(global_label "row1"
 		(shape input)
-		(at 62.23 149.86 180)
+		(at 54.61 149.86 180)
 		(fields_autoplaced yes)
 		(effects
@@
 		)
 		(property "Intersheetrefs" "${INTERSHEET_REFS}"
-			(at 55.4238 149.86 0)
+			(at 47.8038 149.86 0)
 			(effects
 				(font
@@
 					(unit 1)
 				)
+			)
+		)
+	)
+	(symbol
+		(lib_id "Diode:1N4148W")
+		(at 60.96 149.86 0)
+		(unit 1)
+		(exclude_from_sim no)
+		(in_bom yes)
+		(on_board yes)
+		(dnp no)
+		(property "Reference" "D25"
+			(at 61.214 155.956 0)
+			(effects
+				(font
+					(size 1.27 1.27)
+				)
+			)
+		)
+		(property "Value" "1N4148W"
+			(at 61.214 153.162 0)
+			(effects
+				(font
+					(size 1.27 1.27)
+				)
+			)
+		)
+		(property "Footprint" "Diode_SMD:D_SOD-123"
+			(at 60.96 154.305 0)
+			(effects
+				(font
+					(size 1.27 1.27)
+				)
+				(hide yes)
+			)
+		)
+		(property "Datasheet" "https://www.vishay.com/docs/85748/1n4148w.pdf"
+			(at 60.96 149.86 0)
+			(effects
+				(font
+					(size 1.27 1.27)
+				)
+				(hide yes)
+			)
+		)
+		(property "Description" "75V 0.15A Fast Switching Diode, SOD-123"
+			(at 60.96 149.86 0)
+			(effects
+				(font
+					(size 1.27 1.27)
+				)
+				(hide yes)
+			)
+		)
+		(property "Sim.Device" "D"
+			(at 60.96 149.86 0)
+			(effects
+				(font
+					(size 1.27 1.27)
+				)
+				(hide yes)
+			)
+		)
+		(property "Sim.Pins" "1=K 2=A"
+			(at 60.96 149.86 0)
+			(effects
+				(font
+					(size 1.27 1.27)
+				)
+				(hide yes)
+			)
+		)
+		(pin "2"
+		)
+		(pin "1"
+		)
+		(instances
+			(project ""
+				(path "/43cfd488-4c9d-4da2-b703-dd4909c44cb8"
+					(reference "D25")
+					(unit 1)
+				)
